File: boards/core/even_simpler_z80/even_simpler_z80.kicad_sch (KiCad schematic)
At the start: 24 parts, among them J1 Exp. Conn. A, J2 Exp. Conn. B, J3 Power

Commit message: * Working on new powerdistribution method.
Parts:
- removed C2: 0.1uF, Capacitor_THT:C_Disc_D5.0mm_W2.5mm_P2.50mm, symbol Device:C
Changed lines of the file:
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@@
   (title_block
     (title "Even simpler Z80 board")
-    (date "2023-09-05")
-    (rev "1.2")
+    (date "2023-10-28")
+    (rev "1.4")
   )
   (junction (at 87.63 260.985) (diameter 0) (color 0 0 0 0)
@@
   (junction (at 75.565 281.94) (diameter 0) (color 0 0 0 0)
   )
-  (junction (at 123.825 281.94) (diameter 0) (color 0 0 0 0)
-  )
   (junction (at 63.5 281.94) (diameter 0) (color 0 0 0 0)
   )
@@
   )
   (junction (at 39.37 260.985) (diameter 0) (color 0 0 0 0)
-  )
-  (junction (at 123.825 260.985) (diameter 0) (color 0 0 0 0)
   )
   (junction (at 27.305 260.985) (diameter 0) (color 0 0 0 0)
@@
     (stroke (width 0) (type default))
   )
-  (wire (pts (xy 123.825 274.32) (xy 123.825 281.94))
-    (stroke (width 0) (type default))
-  )
   (wire (pts (xy 331.47 107.95) (xy 351.79 107.95))
     (stroke (width 0) (type default))
@@
     (stroke (width 0) (type default))
   )
-  (wire (pts (xy 111.76 281.94) (xy 123.825 281.94))
+  (wire (pts (xy 111.76 281.94) (xy 138.43 281.94))
     (stroke (width 0) (type default))
   )
@@
     (stroke (width 0) (type default))
   )
-  (wire (pts (xy 123.825 266.7) (xy 123.825 260.985))
-    (stroke (width 0) (type default))
-  )
   (wire (pts (xy 180.975 120.015) (xy 171.45 120.015))
     (stroke (width 0) (type default))
@@
     (stroke (width 0) (type default))
   )
-  (wire (pts (xy 111.76 260.985) (xy 123.825 260.985))
+  (wire (pts (xy 111.76 260.985) (xy 138.43 260.985))
     (stroke (width 0) (type default))
   )
@@
     (stroke (width 0) (type default))
   )
-  (wire (pts (xy 123.825 281.94) (xy 138.43 281.94))
-    (stroke (width 0) (type default))
-  )
   (wire (pts (xy 386.08 56.515) (xy 376.555 56.515))
     (stroke (width 0) (type default))
@@
   )
   (wire (pts (xy 138.43 281.94) (xy 153.035 281.94))
-    (stroke (width 0) (type default))
-  )
-  (wire (pts (xy 123.825 260.985) (xy 138.43 260.985))
     (stroke (width 0) (type default))
   )
@@
         (path "/bddfa220-0b4a-4a31-8ec9-ee6ca5aa59a1"
           (reference "C3") (unit 1)
-        )
-      )
-    )
-  )
-  (symbol (lib_id "Device:C") (at 123.825 270.51 0) (unit 1)
-    (in_bom yes) (on_board yes) (dnp no) (fields_autoplaced)
-    (property "Reference" "C2" (at 127 269.24 0)
-      (effects (font (size 1.27 1.27)) (justify left))
-    )
-    (property "Value" "0.1uF" (at 127 271.78 0)
-      (effects (font (size 1.27 1.27)) (justify left))
-    )
-    (property "Footprint" "Capacitor_THT:C_Disc_D5.0mm_W2.5mm_P2.50mm" (at 124.7902 274.32 0)
-      (effects (font (size 1.27 1.27)) hide)
-    )
-    (property "Datasheet" "~" (at 123.825 270.51 0)
-      (effects (font (size 1.27 1.27)) hide)
-    )
-    (pin "1")
-    (pin "2")
-    (instances
-      (project "clock_reset_board"
-        (path "/132edb24-78a1-4238-ad56-1ca9c93ea1ea"
-          (reference "C2") (unit 1)
-        )
-      )
-      (project "even_simpler_z80"
-        (path "/bddfa220-0b4a-4a31-8ec9-ee6ca5aa59a1/4d75357a-4549-4e6f-9c4c-da9ff3091b0f"
-          (reference "C1") (unit 1)
-        )
-        (path "/bddfa220-0b4a-4a31-8ec9-ee6ca5aa59a1"
-          (reference "C9") (unit 1)
         )
       )
@@
       (effects (font (size 1.27 1.27)) (justify right))
     )
-    (pin "B_D7" output (at 171.45 60.325 0)
-      (effects (font (size 1.27 1.27)) (justify right))
-    )
-    (pin "B_D6" output (at 171.45 57.785 0)
-      (effects (font (size 1.27 1.27)) (justify right))
-    )
-    (pin "B_D5" output (at 171.45 55.245 0)
-      (effects (font (size 1.27 1.27)) (justify right))
-    )
-    (pin "B_D1" output (at 171.45 45.085 0)
-      (effects (font (size 1.27 1.27)) (justify right))
-    )
-    (pin "B_D2" output (at 171.45 47.625 0)
-      (effects (font (size 1.27 1.27)) (justify right))
-    )
-    (pin "B_D0" output (at 171.45 42.545 0)
-      (effects (font (size 1.27 1.27)) (justify right))
-    )
-    (pin "B_D3" output (at 171.45 50.165 0)
-      (effects (font (size 1.27 1.27)) (justify right))
-    )
-    (pin "B_D4" output (at 171.45 52.705 0)
-      (effects (font (size 1.27 1.27)) (justify right))
-    )
     (pin "B_A3" output (at 171.45 78.105 0)
       (effects (font (size 1.27 1.27)) (justify right))
@@
       (effects (font (size 1.27 1.27)) (justify left))
     )
-    (instances
+    (pin "B_D6" tri_state (at 171.45 57.785 0)
+      (effects (font (size 1.27 1.27)) (justify right))
+    )
+    (pin "B_D7" tri_state (at 171.45 60.325 0)
+      (effects (font (size 1.27 1.27)) (justify right))
+    )
+    (pin "B_D1" tri_state (at 171.45 45.085 0)
+      (effects (font (size 1.27 1.27)) (justify right))
+    )
+    (pin "B_D2" tri_state (at 171.45 47.625 0)
+      (effects (font (size 1.27 1.27)) (justify right))
+    )
+    (pin "B_D5" tri_state (at 171.45 55.245 0)
+      (effects (font (size 1.27 1.27)) (justify right))
+    )
+    (pin "B_D4" tri_state (at 171.45 52.705 0)
+      (effects (font (size 1.27 1.27)) (justify right))
+    )
+    (pin "B_D3" tri_state (at 171.45 50.165 0)
+      (effects (font (size 1.27 1.27)) (justify right))
+    )
+    (pin "B_D0" tri_state (at 171.45 42.545 0)
+      (effects (font (size 1.27 1.27)) (justify right))
+    )
+    (instances
