File: boards/core/rom_ram_board/rom_ram_board.kicad_pcb (KiCad board)
At the start: 2 copper layers, 95.2 x 95.2 mm, 31 parts, among them J1 Exp. Conn. A, J2 Power, U1 74LS04, U10 62256, U2 74LS30, U3 74LS32, U4 74LS670, U5 28256, U6 74LS367, U7 62256, U8 74LS139, U9 62256

Commit message: * Working on new powerdistribution method.
Parts:
- J2: footprint Connector_IDC:IDC-Header_2x10_P2.54mm_Horizontal -> footprints:TE_171826-4
- moved J2 89.5 mm to (120.1, 105.2), turned to 90 degrees
Connections:
- C1 pad 1: /+5V3 -> /+5V
- C10 pad 1: /+5V3 -> /+5V
- C2 pad 1: /+5V3 -> /+5V
- C3 pad 1: /+5V3 -> /+5V
- C4 pad 1: /+5V3 -> /+5V
- C5 pad 1: /+5V3 -> /+5V
- C6 pad 1: /+5V3 -> /+5V
- C7 pad 1: /+5V3 -> /+5V
- C8 pad 1: /+5V3 -> /+5V
- C9 pad 1: /+5V3 -> /+5V
- CP1 pad 1: /+5V3 -> /+5V
- CP2 pad 1: /+5V3 -> /+5V
- J2 pad 1: /+3.3V -> unconnected-(J2-Pin_1-Pad1)
- J2 pad 2: /+3.3V2 -> /GND
- R1 pad 1: /+5V3 -> /+5V
- U1 pad 14: /+5V3 -> /+5V
- U10 pad 28: /+5V3 -> /+5V
- U2 pad 14: /+5V3 -> /+5V
- U3 pad 14: /+5V3 -> /+5V
- U4 pad 16: /+5V3 -> /+5V
- U5 pad 27: /+5V3 -> /+5V
- U5 pad 28: /+5V3 -> /+5V
- U6 pad 16: /+5V3 -> /+5V
- U7 pad 28: /+5V3 -> /+5V
- U8 pad 16: /+5V3 -> /+5V
- U9 pad 28: /+5V3 -> /+5V
Routing:
- net /+5V: track 0.00 -> 288.6 mm, vias 0 -> 6
- net /+5V3: track 263.5 -> 0.00 mm
- net /GND: track 362.6 -> 345.3 mm, vias 129 -> 128
- net /B_D4: track 181.0 -> 181.7 mm
- net /B_A4: track 186.5 -> 187.1 mm
- net /B_A10: track 144.5 -> 145.1 mm
- net /B_A6: track 171.6 -> 172.1 mm
Other:
- board text added: "+5V"
- board text added: "GND"
- board text added: "NC"
