File: boards/core/rom_ram_board/rom_ram_board.kicad_sch (KiCad schematic)
At the start: 30 parts, among them J1 Exp. Conn. A, J2 Power, U1 74LS04, U10 62256, U2 74LS30, U3 74LS32, U5 28256, U5 74LS670, U6 74LS367, U7 62256, U8 74LS139, U9 62256

Commit message: * Working on new powerdistribution method.
Parts:
- removed J2: Power, Connector_IDC:IDC-Header_2x10_P2.54mm_Horizontal, symbol Connector_Generic:Conn_02x10_Top_Bottom
- added J2: Power, footprints:TE_171826-4, symbol Connector_Generic:Conn_01x04
Connections:
- net +5V3 is gone; now on net +5V: C1.1, C1.1, C2.1, C2.1, C2.1, C2.1, C2.1, C2.1, C2.1, C2.1, CP1.1, CP2.1, R3.1, U1.14 (VCC), U10.28 (VCC), U2.14 (VCC), U3.14 (VCC), U5.16 (VCC), U5.27 (~{WE}), U5.28 (VCC), U6.16 (VCC), U7.28 (VCC), U8.16 (VCC), U9.28 (VCC)
- net +5V: now also J2.4 (Pin_4)
- net GND: now also J2.2 (Pin_2), J2.3 (Pin_3)
- no-connect marks 41 -> 30
