File: boards/msx_compat/msx_rom_ram_board/msx_rom_ram_board.kicad_pcb (KiCad board)
At the start: 2 copper layers, 95.2 x 95.2 mm, 37 parts, among them J1 Exp. Conn. A, J2 Exp. Conn. B, J3 Power, J4 ROM_A18, U1 74LS08, U10 AS6C4008-55PCN, U11 SST39SF040, U2 74LS04, U3 74LS139, U4 74LS30, U5 74LS32, U6 74LS670, U7 74LS670, U8 74LS244, U9 AS6C4008-55PCN

Commit message: * Working on new powerdistribution method.
Parts:
- J3: footprint Connector_IDC:IDC-Header_2x10_P2.54mm_Horizontal -> footprints:TE_171826-4
- moved J3 89.5 mm to (120.1, 105.2), turned to 90 degrees
Connections:
- J3 pad 1: /+3.3V -> unconnected-(J3-Pin_1-Pad1)
- J3 pad 2: /+3.3V2 -> /GND
Routing:
- net /~{B_WR}: track 103.7 -> 158.1 mm, vias 3 -> 5
- net /B_A3: track 151.7 -> 204.5 mm
- net /B_D0: track 134.6 -> 172.2 mm, vias 1 -> 3
- net /B_D3: track 178.6 -> 189.8 mm
- net /B_A8: track 100.0 -> 107.9 mm, vias 2 -> 3
- net /B_A2: track 150.0 -> 156.7 mm, vias 0 -> 1
- net /~{B_M1}: track 131.6 -> 137.8 mm
- net /B_A7: track 196.0 -> 201.5 mm
- net /B_A6: track 178.6 -> 183.3 mm
- net /B_A0: track 108.8 -> 112.6 mm, vias 2 -> 5
- net /B_A14: track 117.9 -> 121.2 mm
- net /+5V: track 405.5 -> 402.8 mm
- net /B_A12: track 129.1 -> 129.8 mm
- net /B_A11: track 77.3 -> 76.7 mm
- net /B_D2: track 145.9 -> 145.5 mm, vias 1 -> 3
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Other:
- board text added: "+5V"
