File: boards/msx_compat/msx_rom_ram_board/msx_rom_ram_board.kicad_sch (KiCad schematic)
At the start: 36 parts, among them J1 Exp. Conn. A, J2 Exp. Conn. B, J3 Power, J4 ROM_A18, U1 74LS08, U10 AS6C4008-55PCN, U11 SST39SF040, U2 74LS04, U3 74LS139, U4 74LS30, U5 74LS32, U5 74LS670, U8 74LS244, U9 AS6C4008-55PCN

Commit message: * Working on new powerdistribution method.
Parts:
- removed J3: Power, Connector_IDC:IDC-Header_2x10_P2.54mm_Horizontal, symbol Connector_Generic:Conn_02x10_Top_Bottom
- added J3: Power, footprints:TE_171826-4, symbol Connector_Generic:Conn_01x04
Connections:
- net +5V: now also J3.4 (Pin_4)
- net GND: now also J3.2 (Pin_2), J3.3 (Pin_3)
- no-connect marks 66 -> 55
