File: boards/msx_compat/ppi_slot_select/ppi_slot_select.kicad_pcb (KiCad board)
At the start: 2 copper layers, 95.2 x 95.2 mm, 27 parts, among them J1 Exp. Conn. A, J2 Exp. Conn. B, J3 Power, J4 GPIO, U1 82C55A_PLCC, U2 74LS00, U3 74LS32, U4 74LS139, U5 74LS138, U6 74LS153

Commit message: * Working on new powerdistribution method.
Parts:
- J3: footprint Connector_IDC:IDC-Header_2x10_P2.54mm_Horizontal -> footprints:TE_171826-4
- R1: value 470 -> 1k
- moved J3 89.5 mm to (120.1, 105.2), turned to 90 degrees
Connections:
- J3 pad 1: /+3.3V -> unconnected-(J3-Pin_1-Pad1)
- J3 pad 2: /+3.3V2 -> /GND
Routing:
- net /+5V: track 262.7 -> 244.6 mm
- net /GND: track 167.3 -> 159.0 mm, vias 58 -> 61
- net /B_A0: track 35.2 -> 35.7 mm
Other:
- board text added: "+5V"
- board text added: "GND"
- board text added: "NC"
