File: boards/msx_compat/ppi_slot_select_expanded/ppi_slot_select_expanded.kicad_pcb (KiCad board)
At the start: 2 copper layers, 95.2 x 95.2 mm, 43 parts, among them J1 Exp. Conn. A, J2 Exp. Conn. B, J3 Power, J4 GPIO, U1 74LS00, U10 74LS153, U11 74LS273, U12 74LS21, U13 74LS153, U14 74LS240, U2 82C55A_PLCC, U3 74LS32, U4 74LS139, U5 74LS21, U6 74LS21, U7 74LS138, U8 74LS04, U9 74LS21

Commit message: * Working on new powerdistribution method.
Parts:
- J3: footprint Connector_IDC:IDC-Header_2x10_P2.54mm_Horizontal -> footprints:TE_171826-4
- moved J3 89.5 mm to (120.1, 105.2), turned to 90 degrees
Connections:
- J3 pad 1: /+3.3V -> unconnected-(J3-Pin_1-Pad1)
- J3 pad 2: /+3.3V2 -> /GND
Routing:
- net /+5V: track 461.6 -> 452.3 mm
- net /~{B_RFSH}: track 126.1 -> 130.9 mm
- net /B_A11: track 38.1 -> 42.0 mm, vias 0 -> 2
- net /B_A7: track 110.9 -> 113.3 mm, vias 0 -> 2
- net /B_A12: track 37.6 -> 39.4 mm
- net /B_A14: track 162.3 -> 162.8 mm
Other:
- board text added: "+5V"
