File: boards/msx_compat/ppi_slot_select_expanded/ppi_slot_select_expanded.kicad_sch (KiCad schematic)
At the start: 42 parts, among them J1 Exp. Conn. A, J2 Exp. Conn. B, J3 Power, J4 GPIO, U1 74LS00, U10 74LS153, U11 74LS273, U12 74LS21, U13 74LS153, U14 74LS240, U2 82C55A_PLCC, U3 74LS32, U4 74LS139, U5 74LS21, U6 74LS21, U7 74LS138, U8 74LS04, U9 74LS21

Commit message: * Working on new powerdistribution method.
Parts:
- removed J3: Power, Connector_IDC:IDC-Header_2x10_P2.54mm_Horizontal, symbol Connector_Generic:Conn_02x10_Top_Bottom
- added J3: Power, footprints:TE_171826-4, symbol Connector_Generic:Conn_01x04
Connections:
- net +5V: now also J3.4 (Pin_4)
- net GND: now also J3.2 (Pin_2), J3.3 (Pin_3)
- no-connect marks 59 -> 48
